File: LedBlinker_Example/LedBlinker_Example.kicad_sch (KiCad schematic)
At the start: 9 parts, among them Q1 2N3904, Q2 2N3906, SW1 SW_Push

Commit message: wip
Parts:
- added J1: Conn_01x02_Pin, symbol Connector:Conn_01x02_Pin
Connections:
- net GND: now also J1.2 (Pin_2)
- net VCC: now also J1.1 (Pin_1)
Other:
- note added: "INPUT:"
- note added: "NPN TRANSISTOR"
- note added: "PNP TRANSISTOR"
